File: CAD/PCB/r1_1/Rev1_1.brd (EAGLE design)
At the start: 99 x 79.2 mm, 40 parts, among them IC1 EEPROM

Commit message: Added C++ support for Pulse Pal 2 Added PCB design files for Pulse Pal 1.1 and 2 Added drivers for Pulse Pal 2 Added microSD file delete option in MATLAB for Pulse Pal 2 Fixed a bug in new trigger syntax in MATLAB Updated license information in file headers Fixed a bug where Win7 COM ports above COM9 wouldn't be recognized in C++
Parts:
- added C5, C6: (no value), SparkFun:CAP-PTH-SMALL
- added JP1: GND, SparkFun-Connectors:1X01
- added JP3: AGND, SparkFun-Connectors:1X01
- added U$7: GNDPLANESHRT, Joshparts2:GNDPLANESHRT
- moved C2 22.3 mm to (58.4, 55.9), turned to 0 degrees
- moved C1 21.8 mm to (62.7, 74.7)
- moved C3 20.5 mm to (74.2, 56.1), turned to 0 degrees
- moved C4 20.3 mm to (74.4, 71.4), turned to 270 degrees
- moved TL084 0.15 mm to (67.6, 63.9), turned to 270 degrees
- turned 10K_RES_ARRAY to 0 degrees
Connections:
- new net AGND: JP3.1, U$3.GND, U$4.GND, U$5.GND, U$6.GND, U$7.AGND
- net GND: now also C5.1, C6.2, JP1.1, U$7.GND; no longer CS.2, MAPLE.GND@2, U$3.GND, U$4.GND, U$5.GND, U$6.GND
- net N$28: now also C5.2
- net N$29: now also C6.1
Routing:
- net GND: track 198.0 -> 0.00 mm
- net N$34: track 71.1 -> 36.0 mm
- net N$1: track 73.2 -> 98.4 mm
- net N$16: track 80.6 -> 103.8 mm, vias 0 -> 1
- net N$33: track 63.7 -> 42.7 mm
- net N$30: track 14.9 -> 31.4 mm, vias 0 -> 1
- net N$42: track 66.1 -> 51.0 mm
- net N$2: track 66.5 -> 80.7 mm, vias 1 -> 2
- net N$35: track 66.5 -> 53.0 mm
- net N$55: track 39.3 -> 27.1 mm, vias 1 -> 0
- net N$8: track 44.9 -> 33.6 mm, vias 1 -> 0
- net N$44: track 21.4 -> 32.7 mm
- net N$17: track 79.2 -> 89.7 mm, vias 0 -> 1
- net N$24: track 17.3 -> 6.87 mm
- net N$41: track 42.9 -> 53.0 mm
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- added copper zone on layer 15, net AGND
- added copper zone on layer 2, net GND
- removed copper zone on layer 16, net GND
Other:
- board text added: "r1.1"
- board text removed: "r1"
