File: CAD/PCB/v3_0/PulsePal_3_0_1.brd (EAGLE design)
At the start: 112 x 98 mm, 55 parts, among them IC1 RS3-0515D, IC2 ACPL-064L-500E, IC3 AD5754RBREZ, IC4 MC79M12CDTRKG, IC5 MC78M12CDTRKG, J1 5227673-1, J2 5227673-1, J3 5227673-1, J4 5227673-1, J5 5227673-1, J6 5227673-1, J7 NHD-2.7-12864WDW3, U1 TEENSY_3.6_DIL

Commit message: -CAD: Updated PCB Design -MATLAB: Updated firmware binaries
Parts:
- removed H1: MOUNT-HOLE3.3, holes:3,3
- removed L2, L3: (no value), WE-CBF:1206
- removed L4: 10μH, SparkFun-Coils:0806
- removed U$6: GNDPLANESHRT, Joshparts2:GNDPLANESHRT
- added C14, C15: 0.1uF, SparkFun-Capacitors:0805
- added C16, C17, C20, C21: 10uf, SparkFun-Capacitors:1206@1
- added C18, C19: 0.01uF, SparkFun-Capacitors:0805
- added C22, C23, C24, C25: 2nF, SparkFun-Capacitors:0805
- added FB1: MPZ2012S221AT000IND_2012_TDK, MPZ2012S221AT000:IND_2012_TDK
- added IC6: ADUM140D1BRZ-RL7R_16_ADI, ADUM140D1BRZ:R_16_ADI
- added R13, R14: 22, Resistor:RESC2012X65
- C10, C11: value 4.7uf -> 1uF; device SparkFun-Capacitors:1206@1 -> SparkFun-Capacitors:0805
- C9: value 4.7uf -> 10uf
- IC4: value MC79M12CDTRKG -> TLV709A33DBVR; device MC79M12CDTRKG:NVD5117PLT4GVF01 -> TLV709A33DBVR:SOT95P280X145-5N
- IC5: value MC78M12CDTRKG -> LT3032IDE-12#PBF; device MC78M12CDTRKG:VREG_MC78M12CDTRKG -> LT3032IDE-12#PBF:LT3032IDE12PBF
- L1: value (none) -> RLS-397IND_LS-397_RCP; device WE-CBF:1206 -> RLS_397:IND_LS-397_RCP
- R1, R2, R3, R4: device SparkFun-Resistors:1206 -> Resistor:RESC2012X65
- R11, R12: value 1k -> 750
- moved C11 18.4 mm to (38.2, 54.9)
- moved IC5 17.8 mm to (47.2, 44.9), turned to 90 degrees
- moved IC4 16.1 mm to (35.0, 52.7), turned to 90 degrees
- moved C10 13.0 mm to (35.0, 48.5), turned to 0 degrees
- moved C9 2.93 mm to (19.6, 49.4), turned to 270 degrees
- moved R2 2.44 mm to (71.8, 52.7)
- moved R4 1.96 mm to (65.7, 52.7), turned to 90 degrees
- moved R3 1.48 mm to (69.8, 52.7)
- moved R1 1.48 mm to (67.7, 52.7)
- moved L1 1.37 mm to (23.1, 49.4), turned to 270 degrees
Connections:
- removed net AGND: C10.1, C11.2, C5.2, C6.2, C7.2, C8.2, IC1.COM, IC3.18, IC3.19, IC3.20, IC3.21, IC4.1, IC5.2_4, J3.GND, J4.GND, J5.GND, J6.GND, U$6.AGND, U1.AGND
- removed net N$41: C9.1, IC1.+VIN, L1.2
- removed net VDD: C7.1, C8.1, IC3.24, IC5.3
- removed net VSS: C5.1, C6.1, IC3.1, IC3.25, IC4.3
- new net +12V: C18.1, C20.1, C7.1, C8.1, IC3.24, IC5.1
- new net +15V: C10.1, IC1.+VOUT, IC4.1, R13.1
- new net -12V: C19.1, C21.1, C5.1, C6.1, IC3.1, IC3.25, IC5.7
- new net -15V: IC1.-VOUT, R14.1
- new net 3V3_ISO: C11.1, C15.2, C3.2, C4.2, IC3.11, IC3.14, IC3.5, IC4.5, IC5.10, IC5.12, IC6.16
- new net D_LDAC: IC6.6, U1.28
- new net D_SCK: IC6.4, U1.13
- new net D_SDA: IC6.5, U1.11
- new net D_SYNC: IC6.3, U1.34/A15
- new net GND_ISO: C10.2, C11.2, C15.1, C16.1, C17.2, C20.2, C21.2, C22.2, C23.2, C24.2, C25.2, C3.1, C4.1, C5.2, C6.2, C7.2, C8.2, IC1.COM, IC3.15, IC3.18, IC3.19, IC3.20, IC3.21, IC4.2, IC5.15, IC5.4, IC5.5, IC6.15, IC6.9, J3.GND, J4.GND, J5.GND, J6.GND, U1.AGND
- new net N$26: C19.2, IC5.11
- net 3V3: now also C14.2, IC6.1; no longer C3.2, C4.2, IC3.11, IC3.14, IC3.5
- net 5V: now also C9.1, FB1.2; no longer L4.1
- net GND: now also C14.1, IC6.2, IC6.7, IC6.8, U1.18/A4; no longer C3.1, C4.1, IC3.15, U$6.GND
- net LED4: now also U1.32/A13; no longer U1.28
- net LED5: now also U1.33/A14; no longer U1.29
- net LED6: now also U1.35/A16; no longer U1.30
- net N$10: now also C23.1
- net N$11: now also C24.1
- net N$12: now also C25.1
- net N$13: now also IC6.14, R2.2; no longer R1.2, U1.11
- net N$14: now also IC6.13; no longer U1.13
- net N$15: now also IC1.+VIN, L1.2; no longer IC1.-VOUT, L3.1
- net N$16: now also C16.2, IC5.16, IC5.6, IC5.9, R14.2; no longer IC1.+VOUT, L2.1
- net N$17: now also IC6.12, R1.2; no longer R2.2, U1.14/A0
- net N$18: now also IC6.11; no longer U1.39/A20
- net N$23: now also C17.1, IC5.14, R13.2; no longer C10.2, IC5.1, L2.2
- net N$24: now also C18.2, IC5.3; no longer C11.1, IC4.2, L3.2
- net N$25: now also FB1.1; no longer L4.2
- net N$9: now also C22.1
- net NAV_B: now also U1.36/A17; no longer U1.34/A15
Routing:
- net 3V3_ISO: track 0.00 -> 101.5 mm, vias 0 -> 6
- net N$17: track 60.7 -> 2.94 mm, vias 1 -> 0
- net GND_ISO: track 0.00 -> 56.3 mm, vias 0 -> 88
- net N$14: track 55.0 -> 2.78 mm
- net VSS: track 49.6 -> 0.00 mm, vias 2 -> 0
- net -12V: track 0.00 -> 46.7 mm, vias 0 -> 2
- net D_SCK: track 0.00 -> 46.6 mm
- net D_SDA: track 0.00 -> 46.4 mm
- net N$13: track 48.8 -> 3.10 mm
- net VDD: track 41.4 -> 0.00 mm, vias 3 -> 0
- net N$18: track 44.2 -> 3.27 mm, vias 1 -> 0
- net LED3: track 35.2 -> 74.8 mm, vias 1 -> 0
- net LED4: track 64.9 -> 91.8 mm
- net D_SYNC: track 0.00 -> 25.8 mm
- net AGND: track 22.4 -> 0.00 mm, vias 10 -> 0
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- added copper zone on layer 1, net -12V
- added copper zone on layer 15, net GND_ISO
- added copper zone on layer 2, net GND_ISO
- removed copper zone on layer 2, net AGND
- removed copper zone on layer 1, net VSS
Other:
- board text added: "rev3.0.1"
- board text removed: "+12V"
- board text removed: "-12V"
- board text removed: "rev3.0.4"
